Commit message: IK Modify

File: src/rascl_description/urdf/rascl.urdf (robot description, URDF)
Before this commit: robot rascl_bot, 8 links, 7 joints
Joints:
- joint lowerarm_joint: limit lower=-1.570796327 upper=1.570796327 effort=100 velocity=1.0 -> lower=-3.141592654 upper=3.141592654 effort=100 velocity=1.0
- joint upperarm_joint: limit lower=-1.570796327 upper=1.570796327 effort=100 velocity=1.0 -> lower=-3.141592654 upper=3.141592654 effort=100 velocity=1.0

Commit message: 坐标系变化

File: src/rascl_description/urdf/rascl.urdf (robot description, URDF)
Before this commit: robot rascl_bot, 8 links, 7 joints
Links:
- added link tcp_link
Joints:
- added joint tcp_fixed_joint: type fixed, parent lowerarm, child tcp_link, origin xyz=0.11616 0.043 0.0179 rpy=0 -1.570796327 0

Commit message: 坐标调节2

File: src/rascl_description/urdf/rascl.urdf (robot description, URDF)
Before this commit: robot rascl_bot, 9 links, 8 joints
Joints:
- joint tcp_fixed_joint: origin xyz=0.11616 0.043 0.0179 rpy=0 -1.570796327 0 -> xyz=0.11478978 0.02881369 0.03193108 rpy=0 -1.570796327 0

Commit message: 改到抓夹中心

File: src/rascl_description/urdf/rascl.urdf (robot description, URDF)
Before this commit: robot rascl_bot, 9 links, 8 joints
Joints:
- joint tcp_fixed_joint: origin xyz=0.11478978 0.02881369 0.03193108 rpy=0 -1.570796327 0 -> xyz=0.13478978 0.02881369 0.03193108 rpy=0 -1.570796327 0

Commit message: spur URDF放宽成2*pi

File: src/rascl_description/urdf/rascl.urdf (robot description, URDF)
Before this commit: robot rascl_bot, 9 links, 8 joints
Joints:
- joint spur_gear_joint: limit lower=-3.1415 upper=3.1415 effort=100 velocity=1.0 -> lower=-6.283185307 upper=6.283185307 effort=100 velocity=1.0

Commit message: 微调坐标

File: src/rascl_description/urdf/rascl.urdf (robot description, URDF)
Before this commit: robot rascl_bot, 9 links, 8 joints
Joints:
- joint tcp_fixed_joint: origin xyz=0.13478978 0.02881369 0.03193108 rpy=0 -1.570796327 0 -> xyz=0.15478978 0.02881369 0.03193108 rpy=0 -1.570796327 0

Commit message: 微调坐标2

File: src/rascl_description/urdf/rascl.urdf (robot description, URDF)
Before this commit: robot rascl_bot, 9 links, 8 joints
Joints:
- joint shoulder_joint: origin xyz=0 0 0.057441 rpy=0 0 0 -> xyz=0 -0.020 0.057441 rpy=0 0 0
- joint tcp_fixed_joint: origin xyz=0.15478978 0.02881369 0.03193108 rpy=0 -1.570796327 0 -> xyz=0.13478978 0.02881369 0.03193108 rpy=0 -1.570796327 0

Commit message: 还原TCP

File: src/rascl_description/urdf/rascl.urdf (robot description, URDF)
Before this commit: robot rascl_bot, 9 links, 8 joints
Joints:
- joint tcp_fixed_joint: origin xyz=0.13478978 0.02881369 0.03193108 rpy=0 -1.570796327 0 -> xyz=0.13916 0 0.0179 rpy=0 -1.570796327 0

Commit message: 坐标系变化

File: src/rascl_description/urdf/rascl.urdf (robot description, URDF)
Before this commit: robot rascl_bot, 9 links, 8 joints
Joints:
- joint shoulder_joint: origin xyz=0 -0.020 0.057441 rpy=0 0 0 -> xyz=0.040 0.020 0.057441 rpy=0 0 0

Commit message: Restore uncompensated CAD coordinate baseline

File: src/rascl_description/urdf/rascl.urdf (robot description, URDF)
Before this commit: robot rascl_bot, 9 links, 8 joints
Links:
- removed link tcp_link
Joints:
- removed joint tcp_fixed_joint
- joint shoulder_joint: origin xyz=0.040 0.020 0.057441 rpy=0 0 0 -> xyz=0 0 0.057441 rpy=0 0 0

Commit message: 修复urdf

File: src/rascl_description/urdf/rascl.urdf (robot description, URDF)
Before this commit: robot rascl_bot, 9 links, 8 joints
Joints:
- joint tcp_fixed_joint: origin xyz=0.13916 0 0.0179 rpy=0 -1.570796327 0 -> xyz=0.170 0 0.0179 rpy=0 -1.570796327 0

Commit message: urdf修改

File: src/rascl_description/urdf/rascl.urdf (robot description, URDF)
Before this commit: robot rascl_bot, 9 links, 8 joints
Joints:
- joint shoulder_joint: origin xyz=0.040 0.020 0.057441 rpy=0 0 0 -> xyz=0 0 0.057441 rpy=0 0 0
